File: Electronic-Remote-Lights-IR.kicad_sch (KiCad schematic)
At the start: 16 parts, among them J1 POWER_PINS, J2 POWER_USB, J3 RELAY, SW1 RESET, U1 VS1338B

Commit message: pcb size optimizations
Parts:
- added H5: MountingHole, MountingHole:MountingHole_2.1mm, symbol Mechanical:MountingHole
Other:
- moved on the sheet: A1, D1, D2, D3, H1, H2, H3, H4, J1, J2, J3, R1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
