File: Electronic-Remote-Lights-IR.kicad_pcb (KiCad board)
At the start: 2 copper layers, 68.6 x 69.2 mm, 16 parts, among them J1 POWER_PINS, J2 POWER_USB, J3 RELAY, SW1 RESET, U1 VS1338B

Commit message: pcb size optimizations
Parts:
- added H5: MountingHole, MountingHole:MountingHole_2.1mm, F.Cu at (104.1, 124.5)
- moved H3 52.5 mm to (131.4, 151.2)
- moved H2 51.8 mm to (131.4, 89.5)
- moved R3 50.8 mm to (106.7, 149.9)
- moved A1 50.8 mm to (81.3, 111.8)
- moved J2 50.8 mm to (107.6, 99.3)
- moved SW1 50.8 mm to (116.6, 114.3)
- moved D1 50.8 mm to (127.0, 127.0)
- moved J1 50.8 mm to (118.1, 96.5)
- moved J3 50.8 mm to (83.8, 96.5)
- moved R1 50.8 mm to (132.1, 109.2)
- moved R2 50.8 mm to (106.7, 144.8)
- moved U1 50.8 mm to (108.0, 137.2)
- moved D2 50.8 mm to (127.0, 137.2)
- moved D3 50.8 mm to (127.0, 147.3)
- moved H4 47.9 mm to (76.2, 151.2)
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Connections:
- A1 pad 23: (no net) -> unconnected-(A1-Pad23)
Routing:
- net GND: track 252.2 -> 252.8 mm
Other:
- board size 68.6 x 69.2 mm -> 62.7 x 69.2 mm

Commit message: rearrange assigned pins
Parts:
- A1: value Arduino Nano v3.0 -> Arduino Nano v3
- H1: value MountingHole -> H1
- H2: value MountingHole -> H2
- H3: value MountingHole -> H3
- H4: value MountingHole -> H4
- J1: value POWER_PINS -> POWER PINS
- J2: value POWER_USB -> POWER USB
Connections:
- J3 pad 1: Net-(A1-Pad26) -> Net-(A1-Pad24)
Routing:
- net Net-(A1-Pad24): track 0.00 -> 37.2 mm
- net Net-(A1-Pad26): track 33.7 -> 0.00 mm
- net GND: track 252.8 -> 247.7 mm
- net Net-(A1-Pad5): track 37.4 -> 36.0 mm
Other:
- board text added: "+"
- board text added: "-"
