File: PCB Diagrams/Electronic-Remote-Lights-IR-v2.kicad_pcb (KiCad board)
At the start: 2 copper layers, 60.9 x 59.7 mm, 16 parts, among them J1 POWER, J2 220V, K1 RELAY, SW1 RESET, U1 VS1338B

Commit message: adding case v2.0 3D model
Parts:
- moved J2 1.27 mm to (82.5, 106.7)
- moved K1 1.27 mm to (95.2, 117.7)
Routing:
- net Net-(A1-Pad5): track 32.1 -> 30.8 mm
- net LINE: track 20.8 -> 20.0 mm
- net GND: track 111.0 -> 111.5 mm
Changed lines of the file:
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@@
   )
   (footprint "TerminalBlock:TerminalBlock_bornier-2_P5.08mm" (layer "F.Cu")
-    (at 81.28 106.68 -90)
+    (at 82.55 106.68 -90)
     (descr "simple 2-pin terminal block, pitch 5.08mm, revamped version of bornier2")
     (tags "terminal block bornier2")
@@
   )
   (footprint "Relay_THT:Relay_SPDT_SANYOU_SRD_Series_Form_C" (layer "F.Cu")
-    (at 93.98 117.72 90)
+    (at 95.25 117.72 90)
     (descr "relay Sanyou SRD series Form C http://www.sanyourelay.ca/public/products/pdf/SRD.pdf")
     (tags "relay Sanyu SRD form C")
@@
     (fp_line (start 16.64 -3.94) (end -1.4 -3.94) (layer "F.SilkS") (width 0.12))
     (fp_line (start 1.27 -1.27) (end -1.4 -1.27) (layer "F.SilkS") (width 0.12))
-    (fp_line (start 1.27 1.27) (end 1.27 -1.27) (layer "F.SilkS") (width 0.12))
     (fp_line (start 13.97 -1.27) (end 13.97 36.83) (layer "F.SilkS") (width 0.12))
     (fp_line (start 1.27 1.27) (end 1.27 36.83) (layer "F.SilkS") (width 0.12))
     (fp_line (start -1.4 1.27) (end -1.4 39.5) (layer "F.SilkS") (width 0.12))
+    (fp_line (start 1.27 1.27) (end 1.27 -1.27) (layer "F.SilkS") (width 0.12))
     (fp_line (start -1.4 39.5) (end 16.64 39.5) (layer "F.SilkS") (width 0.12))
     (fp_line (start 1.27 1.27) (end -1.4 1.27) (layer "F.SilkS") (width 0.12))
@@
   )
   (segment (start 116.84 129.54) (end 120.61 125.77) (width 1.4) (layer "B.Cu") (net 1))
+  (segment (start 89.3 115.77) (end 83.82 121.25) (width 1.4) (layer "B.Cu") (net 1))
   (segment (start 107.952792 124.46) (end 86.36 124.46) (width 1.4) (layer "B.Cu") (net 1))
   (segment (start 78.74 124.46) (end 83.82 124.46) (width 1.4) (layer "B.Cu") (net 1))
@@
   (segment (start 111.76 142.24) (end 119.38 142.24) (width 1.4) (layer "B.Cu") (net 1))
   (segment (start 132.08 142.21) (end 119.41 142.21) (width 1.4) (layer "B.Cu") (net 1))
+  (segment (start 83.82 121.25) (end 83.82 124.46) (width 1.4) (layer "B.Cu") (net 1))
   (segment (start 116.84 139.7) (end 116.84 137.17) (width 1.4) (layer "B.Cu") (net 1))
   (segment (start 109.22 139.7) (end 111.76 142.24) (width 1.4) (layer "B.Cu") (net 1))
-  (segment (start 84.42 119.38) (end 84.42 123.86) (width 1.4) (layer "B.Cu") (net 1))
   (segment (start 109.22 125.727208) (end 107.952792 124.46) (width 1.4) (layer "B.Cu") (net 1))
   (segment (start 116.84 137.17) (end 116.84 129.54) (width 1.4) (layer "B.Cu") (net 1))
   (segment (start 83.82 124.46) (end 86.36 124.46) (width 1.4) (layer "B.Cu") (net 1))
-  (segment (start 84.42 123.86) (end 83.82 124.46) (width 1.4) (layer "B.Cu") (net 1))
-  (segment (start 84.42 119.38) (end 88.03 115.77) (width 1.4) (layer "B.Cu") (net 1))
   (segment (start 116.84 139.7) (end 119.38 142.24) (width 1.4) (layer "B.Cu") (net 1))
   (segment (start 109.22 127) (end 109.22 125.727208) (width 1.4) (layer "B.Cu") (net 1))
@@
   (segment (start 85.1 152.41) (end 78.74 146.05) (width 1.4) (layer "B.Cu") (net 10))
   (segment (start 88.9 152.41) (end 85.1 152.41) (width 1.4) (layer "B.Cu") (net 10))
-  (segment (start 91.44 109.22) (end 93.98 111.76) (width 1.4) (layer "B.Cu") (net 20))
-  (segment (start 86.36 109.22) (end 91.44 109.22) (width 1.4) (layer "B.Cu") (net 20))
-  (segment (start 93.98 111.76) (end 93.98 117.72) (width 1.4) (layer "B.Cu") (net 20))
-  (segment (start 83.82 111.76) (end 86.36 109.22) (width 1.4) (layer "B.Cu") (net 20))
-  (segment (start 81.28 111.76) (end 83.82 111.76) (width 1.4) (layer "B.Cu") (net 20))
+  (segment (start 95.25 117.72) (end 95.25 113.03) (width 1.4) (layer "B.Cu") (net 20))
+  (segment (start 95.25 113.03) (end 91.44 109.22) (width 1.4) (layer "B.Cu") (net 20))
+  (segment (start 86.36 109.22) (end 83.82 111.76) (width 1.4) (layer "B.Cu") (net 20))
+  (segment (start 82.55 111.76) (end 83.82 111.76) (width 1.4) (layer "B.Cu") (net 20))
+  (segment (start 91.44 109.22) (end 86.36 109.22) (width 1.4) (layer "B.Cu") (net 20))
   (segment (start 120.69 130.77) (end 133.24 130.77) (width 1.4) (layer "B.Cu") (net 22))
   (segment (start 119.38 132.08) (end 120.69 130.77) (width 1.4) (layer "B.Cu") (net 22))
@@
   (segment (start 88.9 137.16) (end 83.82 132.08) (width 1.4) (layer "B.Cu") (net 29))
   (segment (start 114.3 121.92) (end 114.3 137.16) (width 1.4) (layer "B.Cu") (net 32))
-  (segment (start 108.15 115.77) (end 100.03 115.77) (width 1.4) (layer "B.Cu") (net 32))
+  (segment (start 101.3 115.77) (end 108.15 115.77) (width 1.4) (layer "B.Cu") (net 32))
   (segment (start 114.3 121.92) (end 108.15 115.77) (width 1.4) (layer "B.Cu") (net 32))
   (segment (start 111.76 127) (end 111.76 137.17) (width 1.4) (layer "B.Cu") (net 33))
-  (segment (start 84.44 103.52) (end 81.28 106.68) (width 1.4) (layer "B.Cu") (net 34))
-  (segment (start 87.98 103.52) (end 84.44 103.52) (width 1.4) (layer "B.Cu") (net 34))
+  (segment (start 89.25 103.52) (end 85.71 103.52) (width 1.4) (layer "B.Cu") (net 34))
+  (segment (start 85.71 103.52) (end 82.55 106.68) (width 1.4) (layer "B.Cu") (net 34))
 )

Commit message: PCB bug fix
Parts:
- added D4: 1N4007, Diode_THT:D_DO-41_SOD81_P10.16mm_Horizontal, F.Cu at (101.6, 119.4)
- added Q1: BC547, Package_TO_SOT_THT:TO-92_Inline_Wide, F.Cu at (114.3, 124.5)
- moved U1 5.08 mm to (111.8, 132.1)
- moved K1 2.84 mm to (96.5, 115.2)
- moved H2 2.84 mm to (133.3, 97.8)
- moved H1 2.54 mm to (78.7, 97.8)
- moved SW1 1.27 mm to (132.0, 130.8)
- moved R1 1.27 mm to (102.9, 132.1)
- moved H3 1.27 mm to (133.3, 152.4)
Connections:
- K1 pad 2: Net-(A1-Pad5) -> Net-(K1-Pad2)
Routing:
- net +5V: track 54.0 -> 94.7 mm
- net Net-(A1-Pad5): track 30.8 -> 13.8 mm
- net Net-(K1-Pad2): track 0.00 -> 16.5 mm
- net GND: track 111.5 -> 119.3 mm
- net Net-(A1-Pad6): track 10.2 -> 5.09 mm
- net NEUT: track 8.01 -> 11.1 mm
- net LINE: track 20.0 -> 18.0 mm
- net Net-(D1-Pad2): track 6.13 -> 6.66 mm
- net Net-(A1-Pad3): track 19.5 -> 19.0 mm
Other:
- board size 60.9 x 59.7 mm -> 62.1 x 62.2 mm

Commit message: PCB component renamed
Parts:
- U1: value VS1338B -> VS1838B
Changed lines of the file:
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@@
   (net 33 "Net-(A1-Pad6)")
   (net 34 "NEUT")
-  (net 35 "Net-(K1-Pad2)")
+  (net 35 "Net-(D4-Pad1)")
   (footprint "MountingHole:MountingHole_2.1mm" (layer "F.Cu")
     (at 133.35 97.79)
@@
       (net 32 "Net-(A1-Pad5)") (pinfunction "B") (pintype "input"))
     (pad "3" thru_hole circle (at 5.08 0 180) (size 1.8 1.8) (drill 0.8) (layers *.Cu *.Mask)
-      (net 35 "Net-(K1-Pad2)") (pinfunction "E") (pintype "passive"))
+      (net 35 "Net-(D4-Pad1)") (pinfunction "E") (pintype "passive"))
     (model "${KICAD6_3DMODEL_DIR}/Package_TO_SOT_THT.3dshapes/TO-92_Inline_Wide.wrl"
       (offset (xyz 0 0 0))
@@
       (effects (font (size 1 1) (thickness 0.15)))
     )
-    (fp_text value "VS1338B" (at 2.54 -2.54) (layer "F.Fab")
+    (fp_text value "VS1838B" (at 2.54 -2.54) (layer "F.Fab")
       (effects (font (size 1 1) (thickness 0.15)))
     )
@@
       (net 20 "LINE") (pintype "passive"))
     (pad "2" thru_hole circle (at 1.95 6.05 180) (size 2.5 2.5) (drill 1) (layers *.Cu *.Mask)
-      (net 35 "Net-(K1-Pad2)") (pintype "passive"))
+      (net 35 "Net-(D4-Pad1)") (pintype "passive"))
     (pad "3" thru_hole circle (at 14.15 6.05 180) (size 3 3) (drill 1.3) (layers *.Cu *.Mask)
       (net 21 "unconnected-(K1-Pad3)") (pintype "no_connect"))
@@
     (fp_line (start 10.16 0) (end 7.68 0) (layer "F.Fab") (width 0.1))
     (pad "1" thru_hole rect (at 0 0 180) (size 1.8 1.8) (drill 0.8) (layers *.Cu *.Mask)
-      (net 35 "Net-(K1-Pad2)") (pinfunction "K") (pintype "passive"))
+      (net 35 "Net-(D4-Pad1)") (pinfunction "K") (pintype "passive"))
     (pad "2" thru_hole circle (at 10.16 0 180) (size 1.8 1.8) (drill 0.8) (layers *.Cu *.Mask)
       (net 1 "GND") (pinfunction "A") (pintype "passive"))

Commit message: update track width to 1.5mm
Parts:
- moved H2 47.3 mm to (174.0, 73.7)
- moved D4 47.3 mm to (142.3, 95.2)
- moved H1 47.3 mm to (119.4, 73.7)
- moved H3 47.3 mm to (174.0, 128.3)
- moved J2 47.3 mm to (123.2, 82.5)
- moved K1 47.3 mm to (137.2, 91.0)
- moved R2 47.3 mm to (124.5, 108.0)
- moved R3 47.3 mm to (119.4, 121.9)
- moved U1 47.3 mm to (152.4, 108.0)
- moved D3 47.3 mm to (119.4, 100.3)
- moved H4 47.3 mm to (119.4, 128.3)
- moved Q1 47.3 mm to (155.0, 100.3)
- moved A1 47.3 mm to (165.1, 113.0)
- moved R1 47.3 mm to (143.5, 108.0)
- moved SW1 47.3 mm to (172.6, 106.6)
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