File: PCB Diagrams/Electronic-Remote-Lights-IR-v2.kicad_sch (KiCad schematic)
At the start: 16 parts, among them J1 POWER, J2 220V, K1 RELAY, SW1 RESET, U1 VS1338B

Commit message: PCB bug fix
Parts:
- added D4: 1N4007, Diode_THT:D_DO-41_SOD81_P10.16mm_Horizontal, symbol Diode:1N4007
- added Q1: BC547, Package_TO_SOT_THT:TO-92_Inline_Wide, symbol Transistor_BJT:BC547
Connections:
- net +5V: now also Q1.1 (C)
- net GND: now also D4.2 (A)
- net at A1.5 (D2): now also Q1.2 (B); no longer K1.2
- new net: D4.1 (K), K1.2, Q1.3 (E)
Other:
- moved on the sheet: D2, D3, K1, R2, R3, U1

Commit message: PCB component renamed
Parts:
- U1: value VS1338B -> VS1838B
Changed lines of the file:
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@@
       (effects (font (size 1.27 1.27)) (justify right))
     )
-    (property "Value" "VS1338B" (id 1) (at 90.17 114.3 0)
+    (property "Value" "VS1838B" (id 1) (at 90.17 114.3 0)
       (effects (font (size 1.27 1.27)) (justify right))
     )
@@
     )
     (path "/4854008c-3227-404e-9125-8acbd6988fad"
-      (reference "U1") (unit 1) (value "VS1338B") (footprint "OptoDevice:Vishay_MINICAST-3Pin")
-    )
-  )
+      (reference "U1") (unit 1) (value "VS1838B") (footprint "OptoDevice:Vishay_MINICAST-3Pin")
+    )
+  )

Commit message: update track width to 1.5mm
Other:
- moved on the sheet: A1, D1, D2, D3, D4, H1, H2, H3, H4, J1, J2, K1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
